File: SLM-VERA.kicad_sch (KiCad schematic)
At the start: 22 parts, among them J1 FH35C-45S-0.3SHW(50), J2 FH35C-45S-0.3SHW(50), J3 GPIO, J4 Conn_01x03_Socket, J5 Conn_01x03_Socket, J6 Conn_01x03_Socket, J7 Conn_01x03_Socket, J8 Conn_01x03_Socket, U1 FODM217D, U2 FODM217D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

Commit message: updated R1-R3 values to 1k on SLM-VERA-004
Parts:
- R1, R2, R3: value 10k -> 1k
Changed lines of the file:
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@@
       (effects (font (size 1.27 1.27)))
     )
-    (property "Value" "10k" (at 86.36 50.8 90)
+    (property "Value" "1k" (at 86.36 50.8 90)
       (effects (font (size 1.27 1.27)))
     )
@@
       (effects (font (size 1.27 1.27)))
     )
-    (property "Value" "10k" (at 86.36 36.83 90)
+    (property "Value" "1k" (at 86.36 36.83 90)
       (effects (font (size 1.27 1.27)))
     )
@@
       (effects (font (size 1.27 1.27)))
     )
-    (property "Value" "10k" (at 86.36 64.77 90)
-      (effects (font (size 1.27 1.27)))
-    )
+    (property "Value" "1k" (at 86.36 64.77 90)
+      (effects (font (size 1.27 1.27)))
+    )
